File: ELW2106AA-breakout-board.kicad_sch (KiCad schematic)
At the start: 28 parts, among them J1 Conn_02x04_Male-custom, U1 TLV61046ADB, U2 XC6206P332MR, U3 TXS0108EPW

Commit message: third revision
Parts:
- C10, C11: symbol Grove - OLED Yellow&Blue Display 0.96 (SSD1315)_V1.0-eagle-import:DISCRETE-SMALL_C-0603 -> Device:C_Small
Connections:
- net +3V3: now also U3.10 (OE)
- net NC: now reaches U3.1 (A1)
- net NC: now also U3.12 (B8), U3.13 (B7), U3.20 (B1), U3.8 (A7), U3.9 (A8)
Changed lines of the file:
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@@
   (junction (at 139.7 41.91) (diameter 0) (color 0 0 0 0)
   )
+  (junction (at 138.43 105.41) (diameter 0) (color 0 0 0 0)
+  )
   (junction (at 41.91 52.07) (diameter 0) (color 0 0 0 0)
   )
@@
     (stroke (width 0) (type default) (color 0 0 0 0))
   )
+  (wire (pts (xy 138.43 105.41) (xy 138.43 115.57))
+    (stroke (width 0) (type default) (color 0 0 0 0))
+  )
   (wire (pts (xy 161.29 36.83) (xy 161.29 49.53))
     (stroke (width 0) (type default) (color 0 0 0 0))
@@
     (stroke (width 0) (type default) (color 0 0 0 0))
   )
-  (wire (pts (xy 137.16 105.41) (xy 146.05 105.41))
+  (wire (pts (xy 137.16 105.41) (xy 138.43 105.41))
     (stroke (width 0) (type default) (color 0 0 0 0))
   )
@@
     (stroke (width 0) (type default) (color 0 0 0 0))
   )
+  (wire (pts (xy 158.75 118.11) (xy 162.56 118.11))
+    (stroke (width 0) (type default) (color 0 0 0 0))
+  )
   (wire (pts (xy 120.65 130.81) (xy 138.43 130.81))
     (stroke (width 0) (type default) (color 0 0 0 0))
@@
     (stroke (width 0) (type default) (color 0 0 0 0))
   )
+  (wire (pts (xy 134.62 133.35) (xy 138.43 133.35))
+    (stroke (width 0) (type default) (color 0 0 0 0))
+  )
   (wire (pts (xy 71.12 52.07) (xy 71.12 41.91))
     (stroke (width 0) (type default) (color 0 0 0 0))
   )
+  (wire (pts (xy 158.75 135.89) (xy 162.56 135.89))
+    (stroke (width 0) (type default) (color 0 0 0 0))
+  )
   (wire (pts (xy 157.48 85.09) (xy 154.94 85.09))
     (stroke (width 0) (type default) (color 0 0 0 0))
@@
     (stroke (width 0) (type default) (color 0 0 0 0))
   )
+  (wire (pts (xy 134.62 118.11) (xy 138.43 118.11))
+    (stroke (width 0) (type default) (color 0 0 0 0))
+  )
   (wire (pts (xy 163.83 49.53) (xy 163.83 36.83))
     (stroke (width 0) (type default) (color 0 0 0 0))
@@
     (stroke (width 0) (type default) (color 0 0 0 0))
   )
+  (wire (pts (xy 134.62 135.89) (xy 138.43 135.89))
+    (stroke (width 0) (type default) (color 0 0 0 0))
+  )
   (wire (pts (xy 168.91 36.83) (xy 175.26 36.83))
     (stroke (width 0) (type default) (color 0 0 0 0))
@@
     (stroke (width 0) (type default) (color 0 0 0 0))
   )
-  (wire (pts (xy 45.72 109.22) (xy 45.72 110.49))
+  (wire (pts (xy 45.72 106.68) (xy 45.72 110.49))
     (stroke (width 0) (type default) (color 0 0 0 0))
   )
@@
     (stroke (width 0) (type default) (color 0 0 0 0))
   )
-  (wire (pts (xy 74.93 110.49) (xy 74.93 109.22))
+  (wire (pts (xy 74.93 110.49) (xy 74.93 106.68))
     (stroke (width 0) (type default) (color 0 0 0 0))
   )
@@
     (stroke (width 0) (type default) (color 0 0 0 0))
   )
+  (wire (pts (xy 138.43 105.41) (xy 146.05 105.41))
+    (stroke (width 0) (type default) (color 0 0 0 0))
+  )
   (wire (pts (xy 148.59 41.91) (xy 148.59 49.53))
     (stroke (width 0) (type default) (color 0 0 0 0))
@@
   )
   (wire (pts (xy 151.13 105.41) (xy 160.02 105.41))
+    (stroke (width 0) (type default) (color 0 0 0 0))
+  )
+  (wire (pts (xy 158.75 133.35) (xy 162.56 133.35))
     (stroke (width 0) (type default) (color 0 0 0 0))
   )
@@
     (effects (font (size 1.778 1.5113)) (justify left bottom))
   )
+  (label "NC" (at 162.56 118.11 0)
+    (effects (font (size 1.27 1.27)) (justify left bottom))
+  )
   (label "OLED_D{slash}C#" (at 121.92 66.04 0)
     (effects (font (size 1.27 1.27)) (justify left bottom))
@@
     (effects (font (size 1.27 1.27)) (justify left bottom))
   )
+  (label "NC" (at 134.62 118.11 0)
+    (effects (font (size 1.27 1.27)) (justify left bottom))
+  )
   (label "FRAME_SYNC" (at 212.09 74.93 0)
     (effects (font (size 1.27 1.27)) (justify left bottom))
@@
     (effects (font (size 1.27 1.27)) (justify left bottom))
   )
+  (label "NC" (at 134.62 133.35 0)
+    (effects (font (size 1.27 1.27)) (justify left bottom))
+  )
   (label "OLED_CS" (at 121.92 68.58 0)
     (effects (font (size 1.27 1.27)) (justify left bottom))
   )
+  (label "NC" (at 162.56 135.89 0)
+    (effects (font (size 1.27 1.27)) (justify left bottom))
+  )
   (label "OLED_D{slash}C#" (at 125.73 125.73 0)
     (effects (font (size 1.27 1.27)) (justify left bottom))
   )
   (label "D{slash}C" (at 162.56 125.73 0)
+    (effects (font (size 1.27 1.27)) (justify left bottom))
+  )
+  (label "NC" (at 162.56 133.35 0)
+    (effects (font (size 1.27 1.27)) (justify left bottom))
+  )
+  (label "NC" (at 134.62 135.89 0)
     (effects (font (size 1.27 1.27)) (justify left bottom))
   )
@@
     (pin "2")
   )
-  (symbol (lib_id "Grove - OLED Yellow&Blue Display 0.96 (SSD1315)_V1.0-eagle-import:DISCRETE-SMALL_C-0603") (at 45.72 105.41 90) (unit 1)
-    (in_bom yes) (on_board yes)
-    (property "Reference" "C10" (id 0) (at 43.18 104.7749 90)
+  (symbol (lib_id "Device:C_Small") (at 45.72 104.14 180) (unit 1)
+    (in_bom yes) (on_board yes)
+    (property "Reference" "C10" (id 0) (at 43.18 102.87 0)
       (effects (font (size 0.889 0.7556)) (justify left))
     )
-    (property "Value" "10uF" (id 1) (at 43.18 106.68 90)
+    (property "Value" "10uF" (id 1) (at 43.18 104.7751 0)
       (effects (font (size 0.889 0.7556)) (justify left))
     )
-    (property "Footprint" "Capacitor_SMD:C_0402_1005Metric" (id 2) (at 45.72 105.41 0)
-      (effects (font (size 1.27 1.27)) hide)
-    )
-    (property "Datasheet" "" (id 3) (at 45.72 105.41 0)
+    (property "Footprint" "Capacitor_SMD:C_0402_1005Metric" (id 2) (at 45.72 104.14 0)
+      (effects (font (size 1.27 1.27)) hide)
+    )
+    (property "Datasheet" "~" (id 3) (at 45.72 104.14 0)
       (effects (font (size 1.27 1.27)) hide)
     )
@@
     (pin "1")
   )
-  (symbol (lib_id "Grove - OLED Yellow&Blue Display 0.96 (SSD1315)_V1.0-eagle-import:DISCRETE-SMALL_C-0603") (at 74.93 105.41 90) (unit 1)
-    (in_bom yes) (on_board yes)
-    (property "Reference" "C11" (id 0) (at 77.47 104.7749 90)
+  (symbol (lib_id "Device:C_Small") (at 74.93 104.14 180) (unit 1)
+    (in_bom yes) (on_board yes)
+    (property "Reference" "C11" (id 0) (at 77.47 102.87 0)
       (effects (font (size 0.889 0.7556)) (justify right))
     )
-    (property "Value" "10uF" (id 1) (at 77.47 106.68 90)
+    (property "Value" "10uF" (id 1) (at 77.47 104.7751 0)
       (effects (font (size 0.889 0.7556)) (justify right))
     )
-    (property "Footprint" "Capacitor_SMD:C_0402_1005Metric" (id 2) (at 74.93 105.41 0)
-      (effects (font (size 1.27 1.27)) hide)
-    )
-    (property "Datasheet" "" (id 3) (at 74.93 105.41 0)
+    (property "Footprint" "Capacitor_SMD:C_0402_1005Metric" (id 2) (at 74.93 104.14 0)
+      (effects (font (size 1.27 1.27)) hide)
+    )
+    (property "Datasheet" "~" (id 3) (at 74.93 104.14 0)
       (effects (font (size 1.27 1.27)) hide)
     )
@@
     (pin "2")
   )
-  (symbol (lib_id "ADP122AUJZ-3.3-R7:+16V") (at 144.78 36.83 0) (unit 1)
+  (symbol (lib_id "+16v:+16V") (at 144.78 36.83 0) (unit 1)
     (in_bom yes) (on_board yes) (fields_autoplaced)
     (property "Reference" "#PWR013" (id 0) (at 144.78 40.64 0)
@@
     (pin "1")
   )
-  (symbol (lib_id "ADP122AUJZ-3.3-R7:+16V") (at 100.33 52.07 0) (unit 1)
+  (symbol (lib_id "+16v:+16V") (at 100.33 52.07 0) (unit 1)
     (in_bom yes) (on_board yes) (fields_autoplaced)
     (property "Reference" "#PWR012" (id 0) (at 100.33 55.88 0)

Commit message: replace TXS0108E with good ol' SN74LVC245
Parts:
- removed C13: 100nF, Capacitor_SMD:C_0402_1005Metric, symbol Device:C_Small
- removed U1: TLV61046ADB, Package_TO_SOT_SMD:SOT-23-6, symbol Regulator_Switching:TLV61046ADB
- removed U3: TXS0108EPW, Package_SO:TSSOP-20_4.4x6.5mm_P0.65mm, symbol Logic_LevelTranslator:TXS0108EPW
- added D1: 1N5819WS, Diode_SMD:D_SOD-323, symbol Diode:1N5819
- added MH1, MH2, MH3, MH4: MountingHole_Pad, custom:MountingHole_2.7mm_M2.5_Custom_Pad, symbol Mechanical:MountingHole_Pad
- added U1: MT3608, Package_TO_SOT_SMD:SOT-23-6, symbol Regulator_Switching:MT3608
- added U3: SN74LVC245ADBRG4, SN74LVC245ADBRG4:SOP65P780X200-20N, symbol SN74LVC245APWR:SN74LVC245APWR
- C10, C11: value 10uF -> 1µF
- C4: value 10µF -> 22µF; footprint Capacitor_SMD:C_0402_1005Metric -> Capacitor_SMD:C_0805_2012Metric
- C8, C9: value 1.0µF -> 1µF
- L1: value 12µH -> 22µH
Connections:
- net +16V: now also D1.1 (K)
- net +3V3: now also U3.20 (VCC)
- net CS: now also U3.6 (A5)
- net D/C: now also U3.4 (A3)
- net GND: now also MH1.1, MH2.1, MH3.1, MH4.1, U1.2 (GND), U3.1 (DIR), U3.10 (GND), U3.11 (B8), U3.12 (B7), U3.13 (B6), U3.19 (~{OE}), U3.7 (A6), U3.8 (A7), U3.9 (A8)
- net MOSI: now also U3.2 (A1)
- net OLED_CS: now also U3.14 (B5)
- net OLED_D/C#: now also U3.16 (B3)
- net OLED_MOSI: now also U3.18 (B1)
- net OLED_RST: now also U3.15 (B4)
- net OLED_SCLK: now also U3.17 (B2)
- net RESET: now also U3.5 (A4)
- net SCLK: now also U3.3 (A2)
- net VCC: now also U1.4 (EN), U1.5 (IN)
- net at R3.2, R4.1: now also U1.3 (FB)
- net at L1.2: now also D1.2 (A), U1.1 (SW)
Other:
- note added: "For compatibility with 5v MCUs which would run SPI at 5v. SSD1362 does not appear to be 5v tolerant on the signal pins. If 3.3V and VCC are the same, it passes through."
- note added: "Reduces voltage to 3.3v (or passes through if <= 3.3v) SSD1362 is designed to run logic between 2.5v and 3.5v"
- note added: "SN74LVC245APWR"
- note added: "Voltage Reduction"
- note removed: "Reduction Voltage"
- moved on the sheet: C10, C11, J1, U2

Commit message: final draft, add jlcpcb information for fabbing/assembly
Parts:
- C1, C10, C11, C2, C3, C8, C9: symbol Device:C_Small -> +16v:C_Small_1uf; LCSC (none) -> C52923
- C4: symbol Device:C_Small -> +16v:C_Small_22uf; LCSC (none) -> C45783
- C5, C6, C7: symbol Device:C_Small -> +16v:C_Small_4.7uf; LCSC (none) -> C1550
- D1: symbol Diode:1N5819 -> +16v:1N5819; LCSC (none) -> C440261
- H1: footprint ELW2106AA:MOLEX_503480-1400 -> Various:AFC24-S14FIA-00; LCSC (none) -> C262682; Note Requires a Futaba ELW2106AA display module -> Footprint is molex connector, requires a Futaba ELW2106AA d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
- L1: symbol Device:L_Small -> +16v:L_Small_22uH; LCSC (none) -> C86821
- MH1, MH2, MH3, MH4: footprint custom:MountingHole_2.7mm_M2.5_Custom_Pad -> custom:MountingHole_2.2mm_M2_Custom_Pad
- R3: symbol Device:R_Small -> +16v:R_Small_1.4M; LCSC (none) -> C270644
- R4: symbol Device:R_Small -> +16v:R_Small_71.5k; LCSC (none) -> C43534
- U1: LCSC (none) -> C7846
- U2: symbol Regulator_Linear:XC6206PxxxMR -> +16v:XC6206P332MR; LCSC (none) -> C479053
- U3: footprint SN74LVC245ADBRG4:SOP65P780X200-20N -> SN74LVC245APWR:SOP65P640X120-20N; JLCPCB C7846 -> (none); LCSC (none) -> C7848
Other:
- note removed: "SN74LVC245APWR"
